Commit message: rostest joint hard limits

File: resources/model.xacro (robot description, xacro)
@@ -45,9 +45,11 @@
         </inertial>
     </link>
-    <joint name="joint1" type="continuous">
+    <!--    Joint 1 has limits, in urdf -->
+    <joint name="joint1" type="revolute">
         <parent link="link1"/>
         <child link="link2"/>
         <origin xyz="0 ${width} ${height1 - axel_offset}" rpy="0 0 0"/>
         <axis xyz="0 1 0"/>
+        <limit effort="30" velocity="1.0" lower="-2.2" upper="0.7" />
         <dynamics damping="0.7"/>
     </joint>
@@ -76,4 +78,5 @@
         </inertial>
     </link>
+    <!--    Joint 2 has no limits in urdf but limits in params-->
     <joint name="joint2" type="continuous">
         <parent link="link2"/>

Commit message: test limits from param

File: resources/model.xacro (robot description, xacro)
@@ -52,4 +52,5 @@
         <axis xyz="0 1 0"/>
         <limit effort="30" velocity="1.0" lower="-2.2" upper="0.7" />
+        <safety_controller k_velocity="10" k_position="15" soft_lower_limit="-2.0" soft_upper_limit="0.5" />
         <dynamics damping="0.7"/>
     </joint>
@@ -78,10 +79,11 @@
         </inertial>
     </link>
-    <!--    Joint 2 has no limits in urdf but limits in params-->
-    <joint name="joint2" type="continuous">
+    <joint name="joint2" type="revolute">
         <parent link="link2"/>
         <child link="link3"/>
         <origin xyz="0 ${width} ${height2 - axel_offset*2}" rpy="0 0 0"/>
         <axis xyz="0 1 0"/>
+        <limit effort="30" velocity="1.0" lower="-2.2" upper="2.2" />
+        <safety_controller k_velocity="10" k_position="15" soft_lower_limit="-2.0" soft_upper_limit="0.5" />
         <dynamics damping="0.7"/>
     </joint>
